Commit message: Update SCARA_JH.urdf

File: Robot_5/scara_robot_description/urdf/SCARA_JH.urdf (robot description, URDF)
Before this commit: robot scara_robot, 5 links, 4 joints
Links:
- link varilla_link: geometry collision cylinder length=0.12 radius=0.012; visual cylinder length=0.3 radius=0.008
Joints:
- joint Union_1_joint: axis 0 -1 0 -> 0 0 1; origin xyz=0.011085 0.129 0 rpy=0 0 0 -> xyz=0.011085 0.0 0.129 rpy=0 0 0.6109
- joint prismatic_joint: axis 0 1 0 -> 0 0 1; limit lower=-0.15 upper=0.0 effort=100.0 velocity=1.0 -> lower=-0.03 upper=0.0 effort=100.0 velocity=1.0; origin xyz=0.00016129 0.185 0.13 rpy=0 0 0 -> xyz=0.00016129 -0.13 0.185 rpy=0 0 0
- joint union_2_joint: axis 0 1 0 -> 0 0 1; origin xyz=0.0032765 0.033 0.12996 rpy=0 0 0 -> xyz=0.0032765 -0.12996 0.033 rpy=0 0 0
- joint world_fixed: origin xyz=0 0 0 rpy=1.5707 0.0 0.0 -> xyz=0 0 0 rpy=0 0 0
